File: TagMod.kicad_pcb (KiCad board)
At the start: 2 copper layers, 21.1 x 27.2 mm, 10 parts, among them J101 Conn_ARM_JTAG_SWD_20, J103 Conn_ARM_JTAG_SWD_10

Commit message: rev b passes drc, ready for fab
Parts:
- added C1: CL21A106KAYNNNE, easyeda2kicad:C0805, F.Cu at (151.7, 97.4)
- added C2: CL10B224KA8NNNC, easyeda2kicad:C0603, F.Cu at (150.9, 100.4)
- added D1: CUS10S30,H3F, easyeda2kicad:SOD-323_L1.8-W1.3-LS2.5-RD, F.Cu at (151.8, 90.9)
- added D2: CUS10S30,H3F, easyeda2kicad:SOD-323_L1.8-W1.3-LS2.5-RD, F.Cu at (149.8, 87.2)
- added J1: Conn_01x03_Pin, Connector_PinHeader_2.54mm:PinHeader_1x03_P2.54mm_Vertical, F.Cu at (146.0, 110.0)
- added R2: 5K1, Resistor_SMD:R_0603_1608Metric, F.Cu at (141.2, 94.2)
- added R3: 5K1, Resistor_SMD:R_0603_1608Metric, F.Cu at (144.3, 94.2)
- added R4: 5K1, Resistor_SMD:R_0603_1608Metric, B.Cu at (150.1, 90.1)
- added R5: 2K7, Resistor_SMD:R_0603_1608Metric, B.Cu at (141.0, 110.3)
- added R6: 10K, Resistor_SMD:R_0603_1608Metric, F.Cu at (148.5, 106.4)
- added R7: 22K7, Resistor_SMD:R_0603_1608Metric, F.Cu at (151.3, 106.6)
- added R8: 6K1, Resistor_SMD:R_0603_1608Metric, F.Cu at (146.0, 106.4)
- added U1: AMS1117-ADJOFC, easyeda2kicad:SOT-89-3_L4.5-W2.5-P1.50-LS4.1-BR-1, F.Cu at (147.8, 96.3)
- added U2: F.0603.00139/P2-0603R1TS2-06T-002, easyeda2kicad:LED0603-RD, F.Cu at (141.0, 110.2)
- added U3: F.0603.00139/P2-0603R1TS2-06T-002, easyeda2kicad:LED0603-RD, F.Cu at (151.7, 86.8)
- added U4: GT-USB-7010ASV, easyeda2kicad:USB-C-SMD_G-SWITCH_GT-USB-7010ASV, F.Cu at (143.8, 89.9)
- R67, R68, R69, R70: moved to B.Cu
- moved R70 9.08 mm to (147.8, 98.2)
- moved R69 5.59 mm to (148.2, 100.1)
- moved J103 3.77 mm to (142.3, 107.1)
- moved R68 3.75 mm to (150.8, 102.5)
- moved G*** 3.40 mm to (146.7, 101.1)
- moved R67 2.57 mm to (150.9, 106.7), turned to 180 degrees
- moved TP102 1.97 mm to (150.7, 87.0)
- moved TP101 0.10 mm to (150.8, 97.2)
Connections:
- J103 pad 6: unconnected-(J103-SWO/TDO-Pad6) -> /VOUT
- J103 pad 7: /nRF52_TX -> /TARGET_RX
- J103 pad 8: /nRF52_RX -> /TARGET_TX
- R69 pad 2: /nRF52_RX -> /TARGET_RX
- R70 pad 1: /nRF52_TX -> /TARGET_TX
Routing:
- net /VOUT: track 0.00 -> 36.1 mm, vias 0 -> 3
- net /USB-VBUS: track 0.00 -> 15.5 mm, vias 0 -> 2
- net /nRF52_RX: track 14.6 -> 0.00 mm
- net /JLINK_RX: track 2.33 -> 16.3 mm, vias 0 -> 1
- net /ADJ: track 0.00 -> 13.4 mm
- net Net-(D1-K): track 0.00 -> 12.3 mm
- net /nRF52_TX: track 10.7 -> 0.00 mm
- net /JLINK_TX: track 2.12 -> 10.3 mm, vias 0 -> 2
- net /TARGET_TX: track 0.00 -> 8.11 mm
- net /SWDIO: track 15.5 -> 23.4 mm, vias 0 -> 2
- net /RESET_N: track 31.0 -> 37.7 mm, vias 1 -> 2
- net /SWCLK: track 15.5 -> 20.8 mm, vias 0 -> 1
- net /TARGET_RX: track 0.00 -> 5.33 mm
- net Net-(J101-VCC/NC): track 6.60 -> 11.4 mm, vias 0 -> 1
- net Net-(U3-K): track 0.00 -> 4.38 mm, vias 0 -> 1
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Other:
- outline, holes or cut-outs redrawn
- board text added: "1V8"
- board text added: "3V3"
- board text added: "Input Power"
- board text added: "Output Power"
- board text added: "Tag Mod"

Commit message: rev b all checks passed
Parts:
- added G***: LOGO, footprints:tc-pins-10mm, B.Cu at (144.3, 89.6)
Other:
- board text removed: "JL RX"
- board text removed: "JL TX"
- board text removed: "TC RX"
- board text removed: "TC TX"
